Commit message: [082026] Adding features to project

File: src/my_robot_normal_description/urdf/mobile_base.xacro (robot description, xacro)
@@ -17,9 +17,10 @@
         <collision>
             <geometry>
-                <box size="${base_lenght} ${base_width} ${base_height}" />
+                <!-- Narrower collision box to avoid any physical contact with the wheels -->
+                <box size="${base_lenght*0.9} ${base_width*0.8} ${base_height*0.8}" />
             </geometry>
             <origin xyz="0 0 ${base_height/2.0}" rpy="0 0 0" />
        </collision>
-        <xacro:box_inertia m="5.0" x="${base_lenght}" y="${base_width}" z="${base_height}"
+        <xacro:box_inertia m="50.0" x="${base_lenght}" y="${base_width}" z="${base_height}"
                            o_xyz="0 0 ${base_height/2.0}" o_rpy="0 0 0" />
     </link>
@@ -35,9 +36,10 @@
             <collision>
                 <geometry>
+                    <!-- IMPORTANT: Use sphere for collision in Gazebo for better steering -->
                     <sphere radius="${wheel_radius}" />
                 </geometry>
                 <origin xyz="0 0 0" rpy="0 0 0" />
             </collision>
-            <xacro:wheel_inertia m="1.0" r="${wheel_radius}" l="${wheel_length}"
+            <xacro:wheel_inertia m="3.0" r="${wheel_radius}" l="${wheel_length}"
                            o_xyz="0 0 0" o_rpy="${pi / 2.0} 0 0" />
         </link>
@@ -72,7 +74,8 @@
         <parent link="base_link" />
         <child link="right_back_wheel_link"/>
-        <origin xyz="${-base_lenght / 2.5} ${-(base_width+wheel_length)/2.0} 0" rpy="0 0 0"/>
+        <origin xyz="${-base_lenght / 2.5} ${-(base_width+wheel_length)/2.0 - 0.01} 0" rpy="0 0 0"/>
         <axis xyz="0 1 0"/>
-        <limit effort="100" velocity="10"/>
+        <limit effort="10000" velocity="10"/>
+        <dynamics damping="0.1" friction="0.1"/>
         <gazebo>
             <provideFeedback>true</provideFeedback>
@@ -82,7 +85,8 @@
         <parent link="base_link" />
         <child link="left_back_wheel_link"/>
-        <origin xyz="${-base_lenght / 2.5} ${(base_width+wheel_length)/2.0} 0" rpy="0 0 0"/>
+        <origin xyz="${-base_lenght / 2.5} ${(base_width+wheel_length)/2.0 + 0.01} 0" rpy="0 0 0"/>
         <axis xyz="0 1 0"/>
-        <limit effort="100" velocity="10"/>
+        <limit effort="10000" velocity="10"/>
+        <dynamics damping="0.1" friction="0.1"/>
         <gazebo>
             <provideFeedback>true</provideFeedback>
@@ -92,7 +96,8 @@
         <parent link="base_link" />
         <child link="right_front_wheel_link"/>
-        <origin xyz="${base_lenght / 2.5} ${-(base_width+wheel_length)/2.0} 0" rpy="0 0 0"/>
+        <origin xyz="${base_lenght / 2.5} ${-(base_width+wheel_length)/2.0 - 0.01} 0" rpy="0 0 0"/>
         <axis xyz="0 1 0"/>
-        <limit effort="100" velocity="10"/>
+        <limit effort="10000" velocity="10"/>
+        <dynamics damping="0.1" friction="0.1"/>
         <gazebo>
             <provideFeedback>true</provideFeedback>
@@ -102,7 +107,8 @@
         <parent link="base_link" />
         <child link="left_front_wheel_link"/>
-        <origin xyz="${base_lenght / 2.5} ${(base_width+wheel_length)/2.0} 0" rpy="0 0 0"/>
+        <origin xyz="${base_lenght / 2.5} ${(base_width+wheel_length)/2.0 + 0.01} 0" rpy="0 0 0"/>
         <axis xyz="0 1 0"/>
-        <limit effort="100" velocity="10"/>
+        <limit effort="10000" velocity="10"/>
+        <dynamics damping="0.1" friction="0.1"/>
         <gazebo>
             <provideFeedback>true</provideFeedback>

File: src/my_robot_normal_description/urdf/mobile_base_gazebo.xacro (robot description, xacro)
@@ -1,52 +1,37 @@
 <?xml version="1.0"?>
 <robot xmlns:xacro="http://www.ros.org/wiki/xacro">
-    <gazebo reference="base_left_back_wheel_link">
-        <mu1 value="0.1"/>
-        <mu2 value="0.1"/>
-    </gazebo>
-    <gazebo reference="base_right_back_wheel_link">
-        <mu1 value="0.1"/>
-        <mu2 value="0.1"/>
-    </gazebo>
-    <gazebo reference="base_left_front_wheel_link">
-        <mu1 value="0.1"/>
-        <mu2 value="0.1"/>
-    </gazebo>
-    <gazebo reference="base_right_front_wheel_link">
-        <mu1 value="0.1"/>
-        <mu2 value="0.1"/>
-    </gazebo>
-    <gazebo>
-        <plugin
-            filename="gz-sim-joint-controller-system"
-            name="gz::sim::systems::JointController">
-            <joint_name>base_left_front_wheel_joint</joint_name>
-            <topic>/base_left_front_wheel_joint/cmd_vel</topic>
-        </plugin>
-    </gazebo>
-    <gazebo>
-        <plugin
-            filename="gz-sim-joint-controller-system"
-            name="gz::sim::systems::JointController">
-            <joint_name>base_right_front_wheel_joint</joint_name>
-            <topic>/base_right_front_wheel_joint/cmd_vel</topic>
-        </plugin>
-    </gazebo>
-    <gazebo>
-        <plugin
-            filename="gz-sim-joint-controller-system"
-            name="gz::sim::systems::JointController">
-            <joint_name>base_left_back_wheel_joint</joint_name>
-            <topic>/base_left_back_wheel_joint/cmd_vel</topic>
-        </plugin>
-    </gazebo>
-    <gazebo>
-        <plugin
-            filename="gz-sim-joint-controller-system"
-            name="gz::sim::systems::JointController">
-            <joint_name>base_right_back_wheel_joint</joint_name>
-            <topic>/base_right_back_wheel_joint/cmd_vel</topic>
-        </plugin>
-    </gazebo>
+    <xacro:macro name="wheel_gazebo" params="reference">
+        <gazebo reference="${reference}">
+            <mu1 value="1.0"/>
+            <!-- mu2 en 0.6 para que el giro sea pesado y no patine -->
+            <mu2 value="0.6"/>
+            <kp value="1000000.0" />
+            <kd value="100.0" />
+            <fdir1 value="1 0 0"/>
+        </gazebo>
+    </xacro:macro>
+    <xacro:wheel_gazebo reference="left_back_wheel_link"/>
+    <xacro:wheel_gazebo reference="right_back_wheel_link"/>
+    <xacro:wheel_gazebo reference="left_front_wheel_link"/>
+    <xacro:wheel_gazebo reference="right_front_wheel_link"/>
+    <xacro:macro name="joint_ctrl" params="joint_name topic">
+        <gazebo>
+            <plugin
+                filename="gz-sim-joint-controller-system"
+                name="gz::sim::systems::JointController">
+                <joint_name>${joint_name}</joint_name>
+                <topic>${topic}</topic>
+                <!-- PID afinado para mover 50kg con suavidad y precisión -->
+                <p_gain>1000.0</p_gain>
+                <i_gain>0.0</i_gain>
+                <d_gain>300.0</d_gain>
+                <max_force>600.0</max_force>
+            </plugin>
+        </gazebo>
+    </xacro:macro>
+    <xacro:joint_ctrl joint_name="base_left_front_wheel_joint" topic="/base_left_front_wheel_joint/cmd_vel"/>
+    <xacro:joint_ctrl joint_name="base_right_front_wheel_joint" topic="/base_right_front_wheel_joint/cmd_vel"/>
+    <xacro:joint_ctrl joint_name="base_left_back_wheel_joint" topic="/base_left_back_wheel_joint/cmd_vel"/>
+    <xacro:joint_ctrl joint_name="base_right_back_wheel_joint" topic="/base_right_back_wheel_joint/cmd_vel"/>
     <gazebo>
         <plugin

File: src/my_robot_normal_description/urdf/my_robot.urdf.xacro (robot description, xacro)
@@ -4,6 +4,5 @@
     <xacro:include filename="mobile_base.xacro"/>
     <xacro:include filename="mobile_base_gazebo.xacro"/>
-    <xacro:include filename="arm.xacro"/>
-    <xacro:include filename="arm_gazebo.xacro"/>
     <xacro:include filename="camera.xacro"/>
+    <xacro:include filename="lidar.xacro"/>
 </robot>

Commit message: 083126 Adding kalman filtering to fuse sensor

File: src/my_robot_normal_description/urdf/mobile_base.xacro (robot description, xacro)
@@ -76,5 +76,5 @@
         <origin xyz="${-base_lenght / 2.5} ${-(base_width+wheel_length)/2.0 - 0.01} 0" rpy="0 0 0"/>
         <axis xyz="0 1 0"/>
-        <limit effort="10000" velocity="10"/>
+        <limit effort="10000" velocity="30"/>
         <dynamics damping="0.1" friction="0.1"/>
         <gazebo>
@@ -87,5 +87,5 @@
         <origin xyz="${-base_lenght / 2.5} ${(base_width+wheel_length)/2.0 + 0.01} 0" rpy="0 0 0"/>
         <axis xyz="0 1 0"/>
-        <limit effort="10000" velocity="10"/>
+        <limit effort="10000" velocity="30"/>
         <dynamics damping="0.1" friction="0.1"/>
         <gazebo>
@@ -98,5 +98,5 @@
         <origin xyz="${base_lenght / 2.5} ${-(base_width+wheel_length)/2.0 - 0.01} 0" rpy="0 0 0"/>
         <axis xyz="0 1 0"/>
-        <limit effort="10000" velocity="10"/>
+        <limit effort="10000" velocity="30"/>
         <dynamics damping="0.1" friction="0.1"/>
         <gazebo>
@@ -109,5 +109,5 @@
         <origin xyz="${base_lenght / 2.5} ${(base_width+wheel_length)/2.0 + 0.01} 0" rpy="0 0 0"/>
         <axis xyz="0 1 0"/>
-        <limit effort="10000" velocity="10"/>
+        <limit effort="10000" velocity="30"/>
         <dynamics damping="0.1" friction="0.1"/>
         <gazebo>

File: src/my_robot_normal_description/urdf/mobile_base_gazebo.xacro (robot description, xacro)
@@ -46,3 +46,15 @@
         </plugin>
     </gazebo>
+    <!-- Ground Truth Odometry Publisher Plugin for Validation -->
+    <gazebo>
+        <plugin
+            filename="gz-sim-odometry-publisher-system"
+            name="gz::sim::systems::OdometryPublisher">
+            <odom_frame>odom</odom_frame>
+            <robot_base_frame>base_footprint</robot_base_frame>
+            <odom_topic>/model/my_robot/odometry</odom_topic>
+            <odom_publish_frequency>50</odom_publish_frequency>
+            <dimensions>2</dimensions>
+        </plugin>
+    </gazebo>
 </robot>

Commit message: 090626 Mecanum control

File: src/my_robot_normal_description/urdf/mobile_base.xacro (robot description, xacro)
@@ -25,45 +25,5 @@
                            o_xyz="0 0 ${base_height/2.0}" o_rpy="0 0 0" />
     </link>
-    <xacro:macro name="wheel_link" params="prefix0 prefix1">
-        <link name="${prefix0}_${prefix1}_wheel_link">
-            <visual>
-                <geometry>
-                    <cylinder radius="${wheel_radius}" length="${wheel_length}" />
-                </geometry>
-                <origin xyz="0 0 0" rpy="${pi / 2.0} 0 0" />
-                <material name="grey" />
-            </visual>
-            <collision>
-                <geometry>
-                    <!-- IMPORTANT: Use sphere for collision in Gazebo for better steering -->
-                    <sphere radius="${wheel_radius}" />
-                </geometry>
-                <origin xyz="0 0 0" rpy="0 0 0" />
-            </collision>
-            <xacro:wheel_inertia m="3.0" r="${wheel_radius}" l="${wheel_length}"
-                           o_xyz="0 0 0" o_rpy="${pi / 2.0} 0 0" />
-        </link>
-    </xacro:macro>
-    <xacro:wheel_link prefix0="right" prefix1="back"/>
-    <xacro:wheel_link prefix0="left" prefix1="back"/>
-    <xacro:wheel_link prefix0="right" prefix1="front"/>
-    <xacro:wheel_link prefix0="left" prefix1="front"/>
-    <!-- <link name="caster_wheel_link">
-        <visual>
-            <geometry>
-                <sphere radius="${wheel_radius/2.0}" />
-            </geometry>
-            <origin xyz="0 0 0" rpy="0 0 0" />
-            <material name="grey" />
-        </visual>
-        <collision>
-            <geometry>
-                <sphere radius="${wheel_radius/2.0}" />
-            </geometry>
-            <origin xyz="0 0 0" rpy="0 0 0" />
-        </collision>
-        <xacro:caster_wheel_inertia m="0.5" r="${wheel_radius/2.0}"
-                           o_xyz="0 0 0" o_rpy="0 0 0" />
-    </link> -->
+    <xacro:include filename="mecanum_wheel.urdf.xacro"/>
     <joint name="base_joint" type="fixed">
         <parent link="base_footprint"/>
@@ -71,47 +31,40 @@
         <origin xyz="0 0 ${wheel_radius}" rpy="0 0 0"/>
     </joint>
-    <joint name="base_right_back_wheel_joint" type="continuous">
-        <parent link="base_link" />
-        <child link="right_back_wheel_link"/>
-        <origin xyz="${-base_lenght / 2.5} ${-(base_width+wheel_length)/2.0 - 0.01} 0" rpy="0 0 0"/>
-        <axis xyz="0 1 0"/>
-        <limit effort="10000" velocity="30"/>
-        <dynamics damping="0.1" friction="0.1"/>
-        <gazebo>
-            <provideFeedback>true</provideFeedback>
-        </gazebo>
-    </joint>
-    <joint name="base_left_back_wheel_joint" type="continuous">
-        <parent link="base_link" />
-        <child link="left_back_wheel_link"/>
-        <origin xyz="${-base_lenght / 2.5} ${(base_width+wheel_length)/2.0 + 0.01} 0" rpy="0 0 0"/>
-        <axis xyz="0 1 0"/>
-        <limit effort="10000" velocity="30"/>
-        <dynamics damping="0.1" friction="0.1"/>
-        <gazebo>
-            <provideFeedback>true</provideFeedback>
-        </gazebo>
-    </joint>
-    <joint name="base_right_front_wheel_joint" type="continuous">
-        <parent link="base_link" />
-        <child link="right_front_wheel_link"/>
-        <origin xyz="${base_lenght / 2.5} ${-(base_width+wheel_length)/2.0 - 0.01} 0" rpy="0 0 0"/>
-        <axis xyz="0 1 0"/>
-        <limit effort="10000" velocity="30"/>
-        <dynamics damping="0.1" friction="0.1"/>
-        <gazebo>
-            <provideFeedback>true</provideFeedback>
-        </gazebo>
-    </joint>
-    <joint name="base_left_front_wheel_joint" type="continuous">
-        <parent link="base_link" />
-        <child link="left_front_wheel_link"/>
-        <origin xyz="${base_lenght / 2.5} ${(base_width+wheel_length)/2.0 + 0.01} 0" rpy="0 0 0"/>
-        <axis xyz="0 1 0"/>
-        <limit effort="10000" velocity="30"/>
-        <dynamics damping="0.1" friction="0.1"/>
-        <gazebo>
-            <provideFeedback>true</provideFeedback>
-        </gazebo>
-    </joint>
+    <!-- Mecanum Wheels with original cylinder visual, but mecanum collision & inertia -->
+    <xacro:mecanum_wheel
+        side="left_front"
+        radius="${wheel_radius}"
+        width="${wheel_length}"
+        pos_x="${base_lenght / 2.5}"
+        pos_y="${(base_width+wheel_length)/2.0 + 0.01}"
+        pos_z="0"
+        mass="3.0"
+    />
+    <xacro:mecanum_wheel
+        side="right_front"
+        radius="${wheel_radius}"
+        width="${wheel_length}"
+        pos_x="${base_lenght / 2.5}"
+        pos_y="${-(base_width+wheel_length)/2.0 - 0.01}"
+        pos_z="0"
+        mass="3.0"
+    />
+    <xacro:mecanum_wheel
+        side="left_back"
+        radius="${wheel_radius}"
+        width="${wheel_length}"
+        pos_x="${-base_lenght / 2.5}"
+        pos_y="${(base_width+wheel_length)/2.0 + 0.01}"
+        pos_z="0"
+        mass="3.0"
+    />
+    <xacro:mecanum_wheel
+        side="right_back"
+        radius="${wheel_radius}"
+        width="${wheel_length}"
+        pos_x="${-base_lenght / 2.5}"
+        pos_y="${-(base_width+wheel_length)/2.0 - 0.01}"
+        pos_z="0"
+        mass="3.0"
+    />
 </robot>

File: src/my_robot_normal_description/urdf/mobile_base_gazebo.xacro (robot description, xacro)
@@ -1,18 +1,5 @@
 <?xml version="1.0"?>
 <robot xmlns:xacro="http://www.ros.org/wiki/xacro">
-    <xacro:macro name="wheel_gazebo" params="reference">
-        <gazebo reference="${reference}">
-            <mu1 value="1.0"/>
-            <!-- mu2 en 0.6 para que el giro sea pesado y no patine -->
-            <mu2 value="0.6"/>
-            <kp value="1000000.0" />
-            <kd value="100.0" />
-            <fdir1 value="1 0 0"/>
-        </gazebo>
-    </xacro:macro>
-    <xacro:wheel_gazebo reference="left_back_wheel_link"/>
-    <xacro:wheel_gazebo reference="right_back_wheel_link"/>
-    <xacro:wheel_gazebo reference="left_front_wheel_link"/>
-    <xacro:wheel_gazebo reference="right_front_wheel_link"/>
+    <!-- Wheel surface friction is configured inside mecanum_wheel.urdf.xacro using fdir1 -->
     <xacro:macro name="joint_ctrl" params="joint_name topic">
         <gazebo>
@@ -22,9 +9,4 @@
                 <joint_name>${joint_name}</joint_name>
                 <topic>${topic}</topic>
-                <!-- PID afinado para mover 50kg con suavidad y precisión -->
-                <p_gain>1000.0</p_gain>
-                <i_gain>0.0</i_gain>
-                <d_gain>300.0</d_gain>
-                <max_force>600.0</max_force>
             </plugin>
         </gazebo>

File: src/my_robot_normal_description/urdf/my_robot.urdf.xacro (robot description, xacro)
@@ -1,4 +1,4 @@
 <?xml version="1.0"?>
-<robot name= "my_robot" xmlns:xacro="http://www.ros.org/wiki/xacro">
+<robot name="my_robot" xmlns:xacro="http://www.ros.org/wiki/xacro" xmlns:gz="http://gazebosim.org/schema">
     <xacro:include filename="common_properties.xacro"/>
     <xacro:include filename="mobile_base.xacro"/>
